Commit message: adding act cameras

File: mani_skill/assets/robots/panda/panda_v2.urdf (robot description, URDF)
Before this commit: robot panda, 15 links, 14 joints
Links:
- added link camera_base_link
- added link camera_link
Joints:
- added joint camera_link_joint: type fixed, parent camera_base_link, child camera_link, origin xyz=0 0.02 0.0115 rpy=0 0 0
- added joint realsense_joint: type fixed, parent panda_hand, child camera_base_link, origin xyz=0.035 0 0.036 rpy=0 -1.5707 3.1415
