Commit message: Created TwoRobotPickCube-v1, PassBottleOver, PlaceInDrawer, DoubleDrawerOpen

File: mani_skill/assets/robots/panda/dual_panda_table.urdf (robot description, URDF)
Before this commit: robot dual_panda_setup, 28 links, 27 joints
Joints:
- joint panda_1_base_joint: origin xyz=0 -0.6 0.025 rpy=0 0 0 -> xyz=-0.4 -0.6 0.025 rpy=0 0 0
- joint panda_2_base_joint: origin xyz=0 0.6 0.025 rpy=0 0 3.14159 -> xyz=-0.4 0.6 0.025 rpy=0 0 3.14159

Commit message: Changes to bimanual environments

File: mani_skill/assets/robots/panda/dual_panda_table.urdf (robot description, URDF)
Before this commit: robot dual_panda_setup, 28 links, 27 joints
Links:
- link table: geometry collision box size=1.2 1.6 0.05; visual mesh filename=table.glb scale=0.8333333333333334 1 1
